File: hardware/kicad/Starbie.kicad_sch (KiCad schematic)
At the start: 0 parts

Commit message: Complete Starbie PCB and manufacturing files
Parts:
- added J1: XIAO-ESP32-C3-SMD, Seeed_Studio_XIAO_Series:XIAO-ESP32-C3-SMD, symbol Seeed_Studio_XIAO_Series:XIAO-ESP32-C3-SMD
- added J2: Conn_01x04, Imported Parts:Display_128x64_096_I2C, symbol Connector_Generic:Conn_01x04
- added J3: MPU6050, Imported Parts:MPU6050_Module, symbol Connector_Generic:Conn_01x08
- added R1: 10k, Resistor_THT:R_Axial_DIN0204_L3.6mm_D1.6mm_P7.62mm_Horizontal, symbol Device:R
- added SW1, SW2: Omron B3F-1000, Button_Switch_THT:SW_TH_Tactile_Omron_B3F-10xx, symbol Switch:SW_Push
- added U1: DHT11, Sensor:Aosong_DHT11_5.5x12.0_P2.54mm, symbol Sensor:DHT11
Connections:
- new net +3V3: J1.12 (3V3_OUT), J2.2 (Pin_2), J3.1 (Pin_1), R1.2, U1.1 (VDD)
- new net BUTTON1: J1.3 (D2), SW1.1
- new net BUTTON2: J1.4 (D3), SW2.1
- new net DHT_DATA: J1.2 (D1), R1.1, U1.2 (DATA)
- new net GND: J1.13 (GND), J2.1 (Pin_1), J3.2 (Pin_2), SW1.2, SW2.2, U1.4 (GND)
- new net I2C_SCL: J1.6 (D5), J2.3 (Pin_3), J3.3 (Pin_3)
- new net I2C_SDA: J1.5 (D4), J2.4 (Pin_4), J3.4 (Pin_4)
- no-connect marks 0 -> 4
